File: doc/hardware/usd-adapter/usd-adapter.sch (KiCad schematic (older format))
At the start: 2 parts, among them J1 usd-plug, P1 CONN_02X04

Commit message: Fix connectors and increase board size on usd-adapter
Parts:
- P1: footprint connectors:strip_2x4_1.27 -> Pin_Headers:Pin_Header_Straight_2x04
Changed lines of the file:
@@
 LIBS:valves
 LIBS:usd-plug
-LIBS:usd-adapter-cache
 EELAYER 25 0
 EELAYER END
@@
 F 0 "P1" H 7000 3450 50  0000 C CNN
 F 1 "CONN_02X04" H 7000 2950 50  0000 C CNN
-F 2 "connectors:strip_2x4_1.27" H 7000 2000 60  0001 C CNN
+F 2 "Pin_Headers:Pin_Header_Straight_2x04" H 7000 2000 60  0001 C CNN
 F 3 "" H 7000 2000 60  0000 C CNN
 	1    7000 3200

Commit message: Change via's shape to oval and check manufacturer requirements
Parts:
- P1: footprint Pin_Headers:Pin_Header_Straight_2x04 -> connectors:PSB_IDC_4x2
Changed lines of the file:
@@
 F 0 "P1" H 7000 3450 50  0000 C CNN
 F 1 "CONN_02X04" H 7000 2950 50  0000 C CNN
-F 2 "Pin_Headers:Pin_Header_Straight_2x04" H 7000 2000 60  0001 C CNN
+F 2 "connectors:PSB_IDC_4x2" H 7000 2000 60  0001 C CNN
 F 3 "" H 7000 2000 60  0000 C CNN
 	1    7000 3200
