File: doc/hardware/main-board/sd-mux.sch (KiCad schematic (older format))
At the start: 48 parts, among them J1 USDCARD, P1 USB_OTG, P10 MKDS 1,5/3, P2 629105136821, P3 61400416021, P4 61400416021, P5 IDC_02X04, P6 IDC_02X04, P7 MKDS 1,5/3, P8 CONN_02X02, P9 CONN_02X02, Q1 IRF7606PBF, Q2 IRF7606PBF, Q3 IRF7606PBF, Q4 IRF7606PBF, Q5 2N7002, Q6 2N7002, Q7 IRF7606PBF, Q8 IRF7606PBF, U1 TS3USB30EDGSR, U2 FT245RL, U3 74AHC1G14, U4 TS3A27518E, U5 74AHC1G14

Commit message: Fix SD card slot, remove SD card power leakage and add power connectors
Parts:
- removed P10, P7: MKDS 1,5/3, footprints:cons_1,5x3, symbol CONN_01X03
- removed P8, P9: CONN_02X02, footprints:PSB_IDC_4x2, symbol CONN_02X02
- added C10, C11: 27p, Capacitors_SMD:C_0805_HandSoldering, symbol C
- added D3, D4: RB751V40T1G, Diodes_SMD:SOD-323, symbol D_Schottky
- added P10, P7: BARREL_JACK, Connect:BARREL_JACK, symbol BARREL_JACK
- added P8: USB_A, footprints:conn_usb_A, symbol USB_A
- added P9: USB_OTG, footprints:conn_usb_B_micro, symbol USB_OTG
- added R12, R13: 4.7K, Resistors_SMD:R_0805_HandSoldering, symbol R
- J1: footprint footprints:microsd_socket -> footprints:HIROSE-MICROSD-DM3AT-SF
- RL1: value G2RK-2 -> G2RK-2-DC5
Connections:
- wire segments 285 -> 296
- no-connect marks 15 -> 20
Other:
- moved on the sheet: D1, D2, J1, P5, P6, Q1, Q2, Q3, Q4, Q5, Q6, R10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
