File: doc/hardware/main-board/sd-mux.sch (KiCad schematic (older format))
At the start: 54 parts, among them J1 USDCARD, P1 USB_OTG, P10 BARREL_JACK, P2 629105136821, P3 61400416021, P4 61400416021, P5 IDC_02X04, P6 IDC_02X04, P7 BARREL_JACK, P8 USB_A, P9 USB_OTG, Q1 IRF7606PBF, Q2 IRF7606PBF, Q3 IRF7606PBF, Q4 IRF7606PBF, Q5 2N7002, Q6 2N7002, Q7 IRF7606PBF, Q8 IRF7606PBF, U1 TS3USB30EDGSR, U2 FT245RL, U3 74AHC1G14, U4 TS3A27518E, U5 74AHC1G14

Commit message: Add USB hub to schematic
Parts:
- removed C1: 27p, Capacitors_SMD:C_0805_HandSoldering, symbol C
- removed P2: 629105136821, footprints:conn_usb_B_micro, symbol USB_OTG
- removed R1: 4.7K, Resistors_SMD:R_0805_HandSoldering, symbol R
- added C12, C15, C16, C17, C19, C20, C21, C22, C23, C24, C26, C28: 100n, Capacitors_SMD:C_0805_HandSoldering, symbol C
- added C13: 1n, Capacitors_SMD:C_0805_HandSoldering, symbol C
- added C14: 1u, Capacitors_SMD:C_0805_HandSoldering, symbol C
- added C18, C25: 18p, Capacitors_SMD:C_0805_HandSoldering, symbol C
- added C27, C29: 10u, Capacitors_SMD:C_0805_HandSoldering, symbol C
- added FB2, FB3: BLM18PG221SN1D, Resistors_SMD:R_0603_HandSoldering, symbol MI0805K400R-10
- added OSC1: ECS-3951M, ECS-3951M:SMD4, symbol ECS-3951M
- added P2: CONN_01X04, Pin_Headers:Pin_Header_Straight_1x04, symbol CONN_01X04
- added R14: 10K, Resistors_SMD:R_0805_HandSoldering, symbol R
- added R15, R21: 1M, Resistors_SMD:R_0805_HandSoldering, symbol R
- added R16, R17, R18, R20: 4.7K, Resistors_SMD:R_0805_HandSoldering, symbol R
- added R19: 9.53K, Resistors_SMD:R_0805_HandSoldering, symbol R
- added U6: TUSB4041IPAPR, TUSB4041IPAPR:QFP50P1200X1200X105-65N, symbol TUSB4041IPAPR
- added U7: TLV73333, TO_SOT_Packages_SMD:SOT-23-5, symbol TLV70233DBV
- added U8: TLV73311, TO_SOT_Packages_SMD:SOT-23-5, symbol TLV70012DDC
- C2: value 27p -> 10u
- P1: footprint footprints:conn_usb_B_micro -> footprints:conn_usb_A
- R2: value 4.7K -> 90.9K
Connections:
- net labels added: 1P1V, 3P3V, USB_DM_DN1, USB_DM_DN2, USB_DP_DN1, USB_DP_DN2, USB_VBUS, XI, XO
- wire segments 296 -> 399
- no-connect marks 20 -> 33
Other:
- note added: "1.1V regulator"
- note added: "24 MHz Crystal"
- note added: "3.3V regulator"
- note added: "FTDI"
- note added: "Port #1 USB hub"
- note added: "Port #2 USB hub"
- note added: "Power relay"
- note added: "USB Hub controller"
- note added: "USB multiplexer"
- note added: "uSD card"
- moved on the sheet: C10, C11, C3, C4, C5, C6, C7, C8, C9, D1, D2, FB1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

Commit message: Add USB hub to the layout
Parts:
- P1: footprint footprints:conn_usb_A -> footprints:conn_usb_B_micro
Connections:
- net labels added: USB_DN1+, USB_DN1-, USB_DN2+, USB_DN2-, USB_MUX1+, USB_MUX1-, USB_MUX2+, USB_MUX2-, USB_UP+, USB_UP-
- net labels removed: USB_DM_DN1, USB_DM_DN2, USB_DP_DN1, USB_DP_DN2
Changed lines of the file:
@@
 F 0 "P1" H 2275 8225 50  0000 C CNN
 F 1 "USB_OTG" H 1950 8550 50  0000 C CNN
-F 2 "footprints:conn_usb_A" V 1900 8250 50  0001 C CNN
+F 2 "footprints:conn_usb_B_micro" V 1900 8250 50  0001 C CNN
 F 3 "" V 1900 8250 50  0000 C CNN
 	1    1950 8350
@@
 XO
 Text Label 3700 7500 0    60   ~ 0
-USB_DP_DN1
+USB_DN1+
 Text Label 3700 7700 0    60   ~ 0
-USB_DP_DN2
+USB_DN2+
 Text Label 3700 7600 0    60   ~ 0
-USB_DM_DN1
+USB_DN1-
 Text Label 3700 7800 0    60   ~ 0
-USB_DM_DN2
+USB_DN2-
 Wire Wire Line
 	6600 7000 6600 7300
@@
 NoConn ~ 4500 6900
 Text Label 2700 2450 0    60   ~ 0
-USB_DP_DN1
+USB_DN1+
 Text Label 2700 2350 0    60   ~ 0
-USB_DM_DN1
+USB_DN1-
 Text Label 2750 12200 0    60   ~ 0
-USB_DM_DN2
+USB_DN2-
 Text Label 2750 12500 0    60   ~ 0
-USB_DP_DN2
+USB_DN2+
 Wire Wire Line
 	2100 6800 1500 6800
@@
 Wire Wire Line
 	2750 8550 2750 9600
+Text Label 2550 8350 0    60   ~ 0
+USB_UP+
+Text Label 2550 8250 0    60   ~ 0
+USB_UP-
+Text Label 5650 12300 0    60   ~ 0
+USB_MUX1+
+Text Label 5650 12200 0    60   ~ 0
+USB_MUX1-
+Text Label 5600 13850 0    60   ~ 0
+USB_MUX2+
+Text Label 5600 13750 0    60   ~ 0
+USB_MUX2-
 $EndSCHEMATC

Commit message: Add missing decoupling capacitor and update fabrication files
Parts:
- added C6: 100n, Capacitors_SMD:C_0805_HandSoldering, symbol C
- renumbered C12 to C1, C16 to C10, C17 to C11, C18 to C12, C19 to C13, C20 to C14, C21 to C15, C22 to C16, C23 to C17, C24 to C18, C25 to C19, C26 to C20, C27 to C21, C28 to C22, C29 to C23, C6 to C24, C7 to C25, C8 to C26, C9 to C27, C10 to C28, C11 to C29, C13 to C3, C14 to C4, C3 to C5, C15 to C7, C4 to C8, C5 to C9, D3 to D2, D4 to D3, D2 to D4, P3 to P2, P4 to P3, P2 to P4, P7 to P5, P5 to P6, P6 to P7, P9 to P8, P8 to P9, Q7 to Q1, Q8 to Q2, Q1 to Q3, Q2 to Q4, Q3 to Q7, Q4 to Q8, R15 to R1, R5 to R10, R3 to R11, R4 to R12, R21 to R13, R6 to R14, R7 to R15, R12 to R16, R8 to R17, R9 to R18, R10 to R19, R13 to R20, R11 to R3, R14 to R4, R16 to R5, R17 to R6, R18 to R7, R19 to R8, R20 to R9, U6 to U3, U5 to U4, U7 to U5, U8 to U6, U3 to U7, U4 to U8
Connections:
- wire segments 399 -> 400

Commit message: Fix crystal on layout
Parts:
- removed OSC1: ECS-3951M, ECS-3951M:SMD4, symbol ECS-3951M
- added X1: CRYSTAL_SMD, Crystals:Crystal_SMD_5032_4Pads, symbol CRYSTAL_SMD
Connections:
- wire segments 400 -> 398
- no-connect marks 33 -> 32
Other:
- moved on the sheet: C12, C19, R13
Changed lines of the file:
@@
 L R R13
 U 1 1 577E2C00
-P 7900 9550
-F 0 "R13" V 7980 9550 50  0000 C CNN
-F 1 "1M" V 7800 9550 50  0000 C CNN
-F 2 "Resistors_SMD:R_0805_HandSoldering" V 7830 9550 50  0001 C CNN
-F 3 "" H 7900 9550 50  0000 C CNN
-	1    7900 9550
+P 7900 9650
+F 0 "R13" V 7980 9650 50  0000 C CNN
+F 1 "1M" V 7800 9650 50  0000 C CNN
+F 2 "Resistors_SMD:R_0805_HandSoldering" V 7830 9650 50  0001 C CNN
+F 3 "" H 7900 9650 50  0000 C CNN
+	1    7900 9650
 	0    -1   -1   0
 $EndComp
@@
 L C C12
 U 1 1 577E2F98
-P 7400 9800
-F 0 "C12" H 7425 9900 50  0000 L CNN
-F 1 "18p" H 7425 9700 50  0000 L CNN
-F 2 "Capacitors_SMD:C_0805_HandSoldering" H 7438 9650 30  0001 C CNN
-F 3 "" H 7400 9800 60  0000 C CNN
-	1    7400 9800
+P 7400 9850
+F 0 "C12" H 7425 9950 50  0000 L CNN
+F 1 "18p" H 7425 9750 50  0000 L CNN
+F 2 "Capacitors_SMD:C_0805_HandSoldering" H 7438 9700 30  0001 C CNN
+F 3 "" H 7400 9850 60  0000 C CNN
+	1    7400 9850
 	1    0    0    -1
 $EndComp
@@
 L C C19
 U 1 1 577E30AE
-P 8400 9800
-F 0 "C19" H 8425 9900 50  0000 L CNN
-F 1 "18p" H 8425 9700 50  0000 L CNN
-F 2 "Capacitors_SMD:C_0805_HandSoldering" H 8438 9650 30  0001 C CNN
-F 3 "" H 8400 9800 60  0000 C CNN
-	1    8400 9800
+P 8400 9850
+F 0 "C19" H 8425 9950 50  0000 L CNN
+F 1 "18p" H 8425 9750 50  0000 L CNN
+F 2 "Capacitors_SMD:C_0805_HandSoldering" H 8438 9700 30  0001 C CNN
+F 3 "" H 8400 9850 60  0000 C CNN
+	1    8400 9850
 	1    0    0    -1
 $EndComp
@@
 $EndComp
 Wire Wire Line
-	7400 9950 7400 10050
+	7400 10000 7400 10050
 Wire Wire Line
 	7400 10050 8400 10050
@@
 	7900 10050 7900 10200
 Wire Wire Line
-	8400 10050 8400 9950
+	8400 10050 8400 10000
 Connection ~ 7900 10050
-$Comp
-L ECS-3951M OSC1
-U 1 1 577E3D9A
-P 7850 8800
-F 0 "OSC1" H 7650 8500 50  0000 L CNN
-F 1 "ECS-3951M" H 7650 9120 50  0000 L CNN
-F 2 "ECS-3951M:SMD4" H 7850 8800 50  0001 L CNN
-F 3 "" H 7850 8800 60  0000 C CNN
-	1    7850 8800
-	0    1    1    0
-$EndComp
-NoConn ~ 7750 9100
-NoConn ~ 7950 9100
-Wire Wire Line
-	7850 9300 7850 9100
-Wire Wire Line
-	7150 9300 7850 9300
-Wire Wire Line
-	7400 9300 7400 9650
-Wire Wire Line
-	7750 9550 7400 9550
-Connection ~ 7400 9550
-Wire Wire Line
-	8050 9100 8050 9300
-Wire Wire Line
-	8050 9300 8700 9300
-Wire Wire Line
-	8400 9300 8400 9650
-Wire Wire Line
-	8050 9550 8400 9550
-Connection ~ 8400 9550
+Wire Wire Line
+	7400 9300 7400 9700
+Wire Wire Line
+	7750 9650 7400 9650
+Connection ~ 7400 9650
+Wire Wire Line
+	8400 9300 8400 9700
+Wire Wire Line
+	8050 9650 8400 9650
+Connection ~ 8400 9650
 Connection ~ 7400 9300
 Connection ~ 8400 9300
@@
 	4850 12850 4850 13000
 Connection ~ 4850 12950
+$Comp
+L CRYSTAL_SMD X1
+U 1 1 57BB80A2
+P 7900 9300
+F 0 "X1" H 7900 9450 50  0000 C CNN
+F 1 "CRYSTAL_SMD" H 7650 9500 50  0001 L CNN
+F 2 "Crystals:Crystal_SMD_5032_4Pads" H 7900 9300 50  0001 C CNN
+F 3 "" H 7900 9300 50  0000 C CNN
+	1    7900 9300
+	1    0    0    -1
+$EndComp
+Wire Wire Line
+	7150 9300 7700 9300
+Wire Wire Line
+	8100 9300 8700 9300
+NoConn ~ 7900 9400
 $EndSCHEMATC

Commit message: Change crystal, swap USB power I/O and wider power tracks to withstand 5A
Parts:
- removed X1: CRYSTAL_SMD, Crystals:Crystal_SMD_5032_4Pads, symbol CRYSTAL_SMD
- added Y1: 24MHz, Crystals:Crystal_HC49-SD_SMD, symbol Crystal
Connections:
- wire segments 398 -> 400
- no-connect marks 32 -> 31
Other:
- moved on the sheet: C28, C29, P8, P9, R16, R20

Commit message: Replace diodes with 0 ohm resistors and testing holes for measuring current leakage
Parts:
- removed D2, D3: RB751V40T1G, Diodes_SMD:SOD-323, symbol D_Schottky
- added R21, R23: 0, Resistors_ThroughHole:Resistor_Horizontal_RM10mm, symbol R
- added R22, R24: 0, Resistors_SMD:R_1210_HandSoldering, symbol R
Connections:
- wire segments 400 -> 408

Commit message: Adapt FTDI's GPIO header to match Adafruit's level shifter
Parts:
- removed P4: CONN_01X04, Pin_Headers:Pin_Header_Straight_1x04, symbol CONN_01X04
- added P4: CONN_01X06, Pin_Headers:Pin_Header_Straight_1x06, symbol CONN_01X06
Connections:
- wire segments 408 -> 412
Other:
- moved on the sheet: C5, FB1, R10, U2

Commit message: Add status LEDs
Parts:
- added D2, D3: LED, LEDs:LED_0603, symbol LED
- added R25, R26: 10K, Resistors_SMD:R_0805_HandSoldering, symbol R
Connections:
- wire segments 412 -> 420
Other:
- moved on the sheet: U7
