File: hardware/main-board/autohat-rig.sch (KiCad schematic (older format))
At the start: 91 parts, among them J1 USDCARD, P1 USB_OTG, P10 BARREL_JACK, P2 61400416021, P3 61400416021, P4 CONN_01X06, P5 BARREL_JACK, P6 IDC_02X04, P7 IDC_02X04, P8 USB_OTG, P9 USB_A, Q1 IRF7606PBF, Q2 IRF7606PBF, Q3 IRF7606PBF, Q4 IRF7606PBF, Q5 2N7002, Q6 2N7002, Q7 IRF7606PBF, Q8 IRF7606PBF, U1 TS3USB30EDGSR, U2 FT245RL, U3 TUSB4041IPAPR, U4 74AHC1G14, U5 TLV73333, U6 TLV73311, U7 74AHC1G14, U8 TS3A27518E, Y1 24MHz

Commit message: Change micro USB socket to through-hole
Parts:
- P1, P8: footprint footprints:conn_usb_B_micro -> footprints:TO_microUSB
Changed lines of the file:
@@
 LIBS:induction
 LIBS:TUSB4041IPAPR
-LIBS:sd-mux-cache
+LIBS:ZX62D-B-5P8
+LIBS:autohat-rig-cache
 EELAYER 25 0
 EELAYER END
@@
 encoding utf-8
 Sheet 1 1
-Title "sd-mux"
-Date "2016-02-26"
-Rev "2"
-Comp "SRPOL"
-Comment1 "Author: Adam Malinowski <a.malinowsk2@partner.samsung.com>"
+Title "autohat-rig"
+Date "2016-12-12"
+Rev "1.0"
+Comp "Resin.io"
+Comment1 "Author: Adam Malinowski <a.malinowsk2@partner.samsung.com> \\n        Tomás Villaseca <tomas@resin.io>"
 Comment2 "Copyright (c) 2016 Samsung Electronics Co., Ltd All Rights Reserved"
 Comment3 ""
@@
 F 0 "P8" H 20525 12675 50  0000 C CNN
 F 1 "USB_OTG" H 20200 13000 50  0000 C CNN
-F 2 "footprints:conn_usb_B_micro" H 20150 12700 50  0001 C CNN
+F 2 "footprints:TO_microUSB" H 20150 12700 50  0001 C CNN
 F 3 "" V 20150 12700 50  0000 C CNN
 	1    20200 12800
@@
 F 0 "P1" H 2275 8225 50  0000 C CNN
 F 1 "USB_OTG" H 1950 8550 50  0000 C CNN
-F 2 "footprints:conn_usb_B_micro" V 1900 8250 50  0001 C CNN
+F 2 "footprints:TO_microUSB" V 1900 8250 50  0001 C CNN
 F 3 "" V 1900 8250 50  0000 C CNN
 	1    1950 8350

Commit message: Fix current leakage
Parts:
- removed Q5, Q6: 2N7002, TO_SOT_Packages_SMD:SOT-23, symbol Q_NMOS_GDS
- removed Q7, Q8: IRF7606PBF, footprints:msoic-8, symbol IRF7606PBF
- removed R17: 10K, Resistors_SMD:R_0805_HandSoldering, symbol R
- removed R21, R23: 0, Resistors_ThroughHole:Resistor_Horizontal_RM10mm, symbol R
- removed R22, R24: 0, Resistors_SMD:R_1210_HandSoldering, symbol R
- removed U7: 74AHC1G14, TO_SOT_Packages_SMD:SOT-23-5, symbol 74AHC1G14
- added C29, C30: 1u, Capacitors_SMD:C_0805_HandSoldering, symbol C
- added C31, C32: 100n, Capacitors_SMD:C_0805_HandSoldering, symbol C
- added R11, R12, R13: 10K, Resistors_SMD:R_0805_HandSoldering, symbol R
- added U7, U8: TPS22860, TPS22860DBVR:SOT95P280X145-6N, symbol TPS22860DBVR
- renumbered C29 to C28, C28 to C33, P9 to P8, P8 to P9, R11 to R14, R12 to R15, R13 to R16, R14 to R17, R15 to R20, R20 to R21, R25 to R22, R26 to R23, R16 to R24, U8 to U9
Connections:
- net labels added: DUT_SEL, TS_SEL
- net labels removed: SOCKET_SEL
- wire segments 420 -> 399
- no-connect marks 31 -> 32
Other:
- note removed: "0 - DUT, 1 - TS"
- moved on the sheet: D2, R22
